Commit message: 将模型文件移动到统一工程下

File: panda_test/robots/dual_panda_example.urdf.xacro (robot description, xacro)
@@ -3,6 +3,6 @@
   <xacro:arg name="arm_id_1" default="panda_1" />
   <xacro:arg name="arm_id_2" default="panda_2" />
-  <xacro:include filename="$(find franka_description)/robots/panda_arm.xacro"/>
-  <xacro:include filename="$(find franka_description)/robots/hand.xacro"/>
+  <xacro:include filename="$(find panda_test)/robots/panda_arm.xacro"/>
+  <xacro:include filename="$(find panda_test)/robots/hand.xacro"/>
   <!-- box shaped table as base for the 2 Pandas -->
   <link name="base">

File: panda_test/robots/hand.xacro (robot description, xacro)
@@ -13,5 +13,5 @@
       <visual>
         <geometry>
-          <mesh filename="package://franka_description/meshes/visual/hand.dae"/>
+          <mesh filename="package://panda_test/meshes/visual/hand.dae"/>
         </geometry>
       </visual>
@@ -56,5 +56,5 @@
       <visual>
         <geometry>
-          <mesh filename="package://franka_description/meshes/visual/finger.dae"/>
+          <mesh filename="package://panda_test/meshes/visual/finger.dae"/>
         </geometry>
       </visual>
@@ -64,5 +64,5 @@
         <origin xyz="0 0 0" rpy="0 0 ${pi}"/>
         <geometry>
-          <mesh filename="package://franka_description/meshes/visual/finger.dae"/>
+          <mesh filename="package://panda_test/meshes/visual/finger.dae"/>
         </geometry>
       </visual>

File: panda_test/robots/panda_arm.urdf.xacro (robot description, xacro)
@@ -7,8 +7,8 @@
   <xacro:unless value="$(arg gazebo)">
     <!-- Create a URDF for a real hardware -->
-    <xacro:include filename="$(find franka_description)/robots/panda_arm.xacro" />
+    <xacro:include filename="$(find panda_test)/robots/panda_arm.xacro" />
     <xacro:panda_arm arm_id="${arm_id}" safety_distance="0.03"/>
     <xacro:if value="$(arg hand)">
-      <xacro:include filename="$(find franka_description)/robots/hand.xacro"/>
+      <xacro:include filename="$(find panda_test)/robots/hand.xacro"/>
       <xacro:hand ns="${arm_id}" rpy="0 0 ${-pi/4}" connected_to="${arm_id}_link8" safety_distance="0.03"/>
     </xacro:if>
@@ -18,7 +18,7 @@
     <xacro:arg name="rpy" default="0 0 0" />
     <!-- Create a simulatable URDF -->
-    <!-- <xacro:include filename="$(find franka_description)/robots/utils.xacro" /> -->
-    <xacro:include filename="$(find franka_description)/robots/panda.transmission.xacro" />
-    <xacro:include filename="$(find franka_description)/robots/panda_gazebo.xacro" />
+    <!-- <xacro:include filename="$(find panda_test)/robots/utils.xacro" /> -->
+    <xacro:include filename="$(find panda_test)/robots/panda.transmission.xacro" />
+    <xacro:include filename="$(find panda_test)/robots/panda_gazebo.xacro" />
     <xacro:panda_arm arm_id="${arm_id}" />
     <xacro:if value="$(arg hand)">

File: panda_test/robots/panda_arm.xacro (robot description, xacro)
@@ -3,5 +3,5 @@
   <!-- safety_distance: Minimum safety distance in [m] by which the collision volumes are expanded and which is enforced during robot motions -->
   <!-- arm_id: Namespace of the panda arm. Serves to differentiate between arms in case of multiple instances. -->
-  <xacro:macro name="panda_arm" params="arm_id:='panda' description_pkg:='franka_description' connected_to:='' xyz:='0 0 0' rpy:='0 0 0' safety_distance:=0">
+  <xacro:macro name="panda_arm" params="arm_id:='panda' description_pkg:='panda_test' connected_to:='' xyz:='0 0 0' rpy:='0 0 0' safety_distance:=0">
     <xacro:unless value="${not connected_to}">
       <joint name="${arm_id}_joint_${connected_to}" type="fixed">

File: panda_test/robots/panda_gazebo.xacro (robot description, xacro)
@@ -15,11 +15,11 @@
         <origin rpy="0 0 0" xyz="0 0 0"/>
         <geometry>
-          <mesh filename="package://franka_description/meshes/visual/link0.dae"/>
-        </geometry>
-      </visual>
-      <collision>
-        <origin rpy="0 0 0" xyz="0 0 0"/>
-        <geometry>
-          <mesh filename="package://franka_description/meshes/collision/link0.stl"/>
+          <mesh filename="package://panda_test/meshes/visual/link0.dae"/>
+        </geometry>
+      </visual>
+      <collision>
+        <origin rpy="0 0 0" xyz="0 0 0"/>
+        <geometry>
+          <mesh filename="package://panda_test/meshes/collision/link0.stl"/>
         </geometry>
       </collision>
@@ -41,11 +41,11 @@
         <origin rpy="0 0 0" xyz="0 0 0"/>
         <geometry>
-          <mesh filename="package://franka_description/meshes/visual/link1.dae"/>
-        </geometry>
-      </visual>
-      <collision>
-        <origin rpy="0 0 0" xyz="0 0 0"/>
-        <geometry>
-          <mesh filename="package://franka_description/meshes/collision/link1.stl"/>
+          <mesh filename="package://panda_test/meshes/visual/link1.dae"/>
+        </geometry>
+      </visual>
+      <collision>
+        <origin rpy="0 0 0" xyz="0 0 0"/>
+        <geometry>
+          <mesh filename="package://panda_test/meshes/collision/link1.stl"/>
         </geometry>
       </collision>
@@ -75,11 +75,11 @@
         <origin rpy="0 0 0" xyz="0 0 0"/>
         <geometry>
-          <mesh filename="package://franka_description/meshes/visual/link2.dae"/>
-        </geometry>
-      </visual>
-      <collision>
-        <origin rpy="0 0 0" xyz="0 0 0"/>
-        <geometry>
-          <mesh filename="package://franka_description/meshes/collision/link2.stl"/>
+          <mesh filename="package://panda_test/meshes/visual/link2.dae"/>
+        </geometry>
+      </visual>
+      <collision>
+        <origin rpy="0 0 0" xyz="0 0 0"/>
+        <geometry>
+          <mesh filename="package://panda_test/meshes/collision/link2.stl"/>
         </geometry>
       </collision>
@@ -109,11 +109,11 @@
         <origin rpy="0 0 0" xyz="0 0 0"/>
         <geometry>
-          <mesh filename="package://franka_description/meshes/visual/link3.dae"/>
-        </geometry>
-      </visual>
-      <collision>
-        <origin rpy="0 0 0" xyz="0 0 0"/>
-        <geometry>
-          <mesh filename="package://franka_description/meshes/collision/link3.stl"/>
+          <mesh filename="package://panda_test/meshes/visual/link3.dae"/>
+        </geometry>
+      </visual>
+      <collision>
+        <origin rpy="0 0 0" xyz="0 0 0"/>
+        <geometry>
+          <mesh filename="package://panda_test/meshes/collision/link3.stl"/>
         </geometry>
       </collision>
@@ -143,11 +143,11 @@
         <origin rpy="0 0 0" xyz="0 0 0"/>
         <geometry>
-          <mesh filename="package://franka_description/meshes/visual/link4.dae"/>
-        </geometry>
-      </visual>
-      <collision>
-        <origin rpy="0 0 0" xyz="0 0 0"/>
-        <geometry>
-          <mesh filename="package://franka_description/meshes/collision/link4.stl"/>
+          <mesh filename="package://panda_test/meshes/visual/link4.dae"/>
+        </geometry>
+      </visual>
+      <collision>
+        <origin rpy="0 0 0" xyz="0 0 0"/>
+        <geometry>
+          <mesh filename="package://panda_test/meshes/collision/link4.stl"/>
         </geometry>
       </collision>
@@ -177,11 +177,11 @@
         <origin rpy="0 0 0" xyz="0 0 0"/>
         <geometry>
-          <mesh filename="package://franka_description/meshes/visual/link5.dae"/>
-        </geometry>
-      </visual>
-      <collision>
-        <origin rpy="0 0 0" xyz="0 0 0"/>
-        <geometry>
-          <mesh filename="package://franka_description/meshes/collision/link5.stl"/>
+          <mesh filename="package://panda_test/meshes/visual/link5.dae"/>
+        </geometry>
+      </visual>
+      <collision>
+        <origin rpy="0 0 0" xyz="0 0 0"/>
+        <geometry>
+          <mesh filename="package://panda_test/meshes/collision/link5.stl"/>
         </geometry>
       </collision>
@@ -211,11 +211,11 @@
         <origin rpy="0 0 0" xyz="0 0 0"/>
         <geometry>
-          <mesh filename="package://franka_description/meshes/visual/link6.dae"/>
-        </geometry>
-      </visual>
-      <collision>
-        <origin rpy="0 0 0" xyz="0 0 0"/>
-        <geometry>
-          <mesh filename="package://franka_description/meshes/collision/link6.stl"/>
+          <mesh filename="package://panda_test/meshes/visual/link6.dae"/>
+        </geometry>
+      </visual>
+      <collision>
+        <origin rpy="0 0 0" xyz="0 0 0"/>
+        <geometry>
+          <mesh filename="package://panda_test/meshes/collision/link6.stl"/>
         </geometry>
       </collision>
@@ -245,11 +245,11 @@
         <origin rpy="0 0 0" xyz="0 0 0"/>
         <geometry>
-          <mesh filename="package://franka_description/meshes/visual/link7.dae"/>
-        </geometry>
-      </visual>
-      <collision>
-        <origin rpy="0 0 0" xyz="0 0 0"/>
-        <geometry>
-          <mesh filename="package://franka_description/meshes/collision/link7.stl"/>
+          <mesh filename="package://panda_test/meshes/visual/link7.dae"/>
+        </geometry>
+      </visual>
+      <collision>
+        <origin rpy="0 0 0" xyz="0 0 0"/>
+        <geometry>
+          <mesh filename="package://panda_test/meshes/collision/link7.stl"/>
         </geometry>
       </collision>
@@ -288,5 +288,5 @@
   </xacro:macro>
   <xacro:macro name="hand" params="connected_to:='' ns:='' xyz:='0 0 0' rpy:='0 0 0'">
-    <xacro:include filename="$(find franka_description)/robots/utils.xacro"/>
+    <xacro:include filename="$(find panda_test)/robots/utils.xacro"/>
     <xacro:unless value="${connected_to == ''}">
       <joint name="${ns}_hand_joint" type="fixed">
@@ -299,5 +299,5 @@
       <visual>
         <geometry>
-          <mesh filename="package://franka_description/meshes/visual/hand.dae"/>
+          <mesh filename="package://panda_test/meshes/visual/hand.dae"/>
         </geometry>
       </visual>
@@ -320,5 +320,5 @@
       <visual>
         <geometry>
-          <mesh filename="package://franka_description/meshes/visual/finger.dae"/>
+          <mesh filename="package://panda_test/meshes/visual/finger.dae"/>
         </geometry>
       </visual>
@@ -341,5 +341,5 @@
         <origin xyz="0 0 0" rpy="0 0 ${pi}"/>
         <geometry>
-          <mesh filename="package://franka_description/meshes/visual/finger.dae"/>
+          <mesh filename="package://panda_test/meshes/visual/finger.dae"/>
         </geometry>
       </visual>
