Commit message: 解决一些规划执行过程中的问题

File: panda_test/robots/panda.transmission.xacro (robot description, xacro)
@@ -1,5 +1,5 @@
 <?xml version="1.0"?>
 <robot xmlns:xacro="http://www.ros.org/wiki/xacro">
-  <xacro:macro name="panda_arm" params="arm_id:='panda'">
+  <xacro:macro name="panda_arm_transmission" params="arm_id:='panda'">
     <transmission name="${arm_id}_tran_1">
         <type>transmission_interface/SimpleTransmission</type>
@@ -72,5 +72,5 @@
         </actuator>
     </transmission>
-    <transmission name="${arm_id}_tran_8">
+    <!-- <transmission name="${arm_id}_tran_8">
         <type>transmission_interface/SimpleTransmission</type>
         <joint name="${arm_id}_joint8">
@@ -81,5 +81,5 @@
             <mechanicalReduction>1</mechanicalReduction>
         </actuator>
-    </transmission>
+    </transmission> -->
   </xacro:macro>
 </robot>

File: panda_test/robots/panda_arm.urdf.xacro (robot description, xacro)
@@ -21,4 +21,5 @@
     <xacro:include filename="$(find panda_test)/robots/panda.transmission.xacro" />
     <xacro:include filename="$(find panda_test)/robots/panda_gazebo.xacro" />
+    <xacro:panda_arm_transmission arm_id="${arm_id}" />
     <xacro:panda_arm arm_id="${arm_id}" />
     <xacro:if value="$(arg hand)">
@@ -34,5 +35,5 @@
       <child  link="${arm_id}_link0" />
     </joint>
-    <xacro:gazebo-joint joint="${arm_id}_joint1" transmission="hardware_interface/EffortJointInterface" />
+    <!-- <xacro:gazebo-joint joint="${arm_id}_joint1" transmission="hardware_interface/EffortJointInterface" />
     <xacro:gazebo-joint joint="${arm_id}_joint2" transmission="hardware_interface/EffortJointInterface" />
     <xacro:gazebo-joint joint="${arm_id}_joint3" transmission="hardware_interface/EffortJointInterface" />
@@ -40,5 +41,5 @@
     <xacro:gazebo-joint joint="${arm_id}_joint5" transmission="hardware_interface/EffortJointInterface" />
     <xacro:gazebo-joint joint="${arm_id}_joint6" transmission="hardware_interface/EffortJointInterface" />
-    <xacro:gazebo-joint joint="${arm_id}_joint7" transmission="hardware_interface/EffortJointInterface" />
+    <xacro:gazebo-joint joint="${arm_id}_joint7" transmission="hardware_interface/EffortJointInterface" /> -->
     <!-- <xacro:transmission-franka-state arm_id="${arm_id}" />
     <xacro:transmission-franka-model arm_id="${arm_id}"
